Commit message: Add model part pressure sensor

File: urdf/zeabus.urdf (robot description, URDF)
Before this commit: robot zeabus, 7 links, 6 joints
Links:
- added link sensor_pressure
Joints:
- added joint base_link_to_sensor_pressure: type fixed, parent base_link, child sensor_pressure, origin xyz=-0.55 0 0 rpy=0 0 0

Commit message: Finish

File: urdf/zeabus.urdf (robot description, URDF)
Before this commit: robot zeabus, 8 links, 7 joints
Joints:
- joint base_link_to_sensor_imu: origin xyz=0.16 0 0 rpy=0 0 ${-PI/2} -> xyz=0.16 0 0 rpy=0 0 ${-PI}
- joint sensor_imu_to_sensor_imu_NED: origin xyz=0 0 0 rpy=${PI} 0 ${-PI/2} -> xyz=0 0 0 rpy=${PI} 0 ${PI/2}

Commit message: Make it correct?

File: urdf/zeabus.urdf (robot description, URDF)
Before this commit: robot zeabus, 8 links, 7 joints
Joints:
- joint bottom_camera_to_optical_frame: origin xyz=0 0 0 rpy=${PI / 2} 0 ${ PI / -2} -> xyz=0 0 0 rpy=${PI / -2} 0 ${ PI / -2}
- joint front_camera_to_optical_frame: origin xyz=0 0 0 rpy=${PI / 2} 0 ${ PI / -2} -> xyz=0 0 0 rpy=${PI / -2} 0 ${ PI / -2}

Commit message: Add translation to bottom camera

File: urdf/zeabus.urdf (robot description, URDF)
Before this commit: robot zeabus, 8 links, 7 joints
Joints:
- joint base_link_bottom_camera: origin xyz=0.26 0 0 rpy=0 ${PI / 2 } 0 -> xyz=0.26 0 -0.1 rpy=0 ${PI / 2 } 0

Commit message: Update model

File: urdf/zeabus.urdf (robot description, URDF)
Before this commit: robot zeabus, 8 links, 7 joints
Links:
- link base_link: geometry visual mesh filename=package://zeabus_model/stl/zeabus.stl scale=0.001 0.001 0.001
